File: alu.kicad_pcb (KiCad board)
At the start: 2 copper layers, 100 x 100 mm, 119 parts, among them J0 640-USB4970-00-A, Q0 DMG2302U-7, Q1 DMG2302U-7, Q2 DMG2302U-7, Q3 DMG2302U-7, Q4 DMG2302U-7, Q5 DMG2302U-7, SW0 418127270904, SW1 418127270904, SW2 418127270904, U0 SN74LS08N, U1 SN74HC86N, U10 SN74LVC1G32DBVR, U11 SN74LS08N, U12 SN74LS08N, U13 CD74HCT32E, U14 CD74HCT32E, U2 SN74HC86N, U3 SN74LS08N, U4 SN74LS08N, U5 CD74HCT32E, U6 SN74LS08N, U7 SN74LS08N, U8 SN74HC86N, U9 SN74LS08N

Commit message: fix: chores pcb
Parts:
- moved D6 1.33 mm to (149.7, 132.9)
- moved D7 1.33 mm to (149.7, 136.9)
- moved D4 1.33 mm to (149.7, 125.0)
- moved D5 1.33 mm to (149.7, 128.7)
- moved D1 1.31 mm to (149.8, 109.5)
- moved D3 1.26 mm to (149.8, 117.8)
- moved D0 1.07 mm to (149.9, 106.2)
- moved D2 0.95 mm to (150.0, 102.2)
Routing:
- net Net-(D3-A): track 5.63 -> 4.05 mm
- net Net-(D1-A): track 4.92 -> 3.51 mm
- net Net-(D4-A): track 5.86 -> 4.56 mm
- net Net-(D7-A): track 6.21 -> 4.91 mm
- net Net-(D6-A): track 6.21 -> 4.91 mm
- net Net-(D0-A): track 4.71 -> 3.57 mm
- net Net-(D2-A): track 5.21 -> 4.21 mm
- net Net-(D5-A): track 5.59 -> 4.68 mm
- net MUL: track 152.1 -> 152.7 mm
- net /binary-decoder/IN_OP2: track 77.9 -> 78.5 mm
- net Net-(Q1-D): track 38.2 -> 38.8 mm
- net OUT_MUL_3: track 41.7 -> 41.1 mm
