File: alu.kicad_pcb (KiCad board)
At the start: 2 copper layers, 100 x 100 mm, 119 parts, among them J0 640-USB4970-00-A, Q0 DMG2302U-7, Q1 DMG2302U-7, Q2 DMG2302U-7, Q3 DMG2302U-7, Q4 DMG2302U-7, Q5 DMG2302U-7, SW0 418127270904, SW1 418127270904, SW2 418127270904, U0 SN74LS08N, U1 SN74HC86N, U10 SN74LVC1G32DBVR, U11 SN74LS08N, U12 SN74LS08N, U13 CD74HCT32E, U14 CD74HCT32E, U2 SN74HC86N, U3 SN74LS08N, U4 SN74LS08N, U5 CD74HCT32E, U6 SN74LS08N, U7 SN74LS08N, U8 SN74HC86N, U9 SN74LS08N

Commit message: feat: v1
Parts:
- removed the G*** at (61.0, 139.5)
- added G***: LOGO, LOGO, F.Cu at (60.5, 138.5)
- added G***: LOGO, LOGO, B.Cu at (143.5, 136.0)
- added G***: LOGO, LOGO, B.Cu at (62.0, 101.0)
- added G***: LOGO, LOGO, B.Cu at (144.3, 107.0)
- C0, C10, C11, C12, C13, C14, C2, C3, C4, C5, C6, C7, C8, C9: value C_Small -> 100nF
- C1: value 885012106031 -> 10uF
- R0, R1, R10, R14, R2, R3, R4, R5, R6, R7, R8, R9: value CRG0603J10K - 3399584 -> 10kΩ
- R11, R12, R13, R17, R18, R19, R20, R21: value RC0603FR-07220RL -> 220Ω
- R15, R16: value RC0603JR-075K1L -> 5.1kΩ
- moved OUT_2 2.66 mm to (135.0, 137.0)
- moved OUT_1 2.30 mm to (135.0, 129.0)
- moved OUT_0 2.30 mm to (135.0, 123.8)
- moved OUT_3 2.30 mm to (135.0, 133.5)
- moved IN_B2 1.70 mm to (66.0, 111.5)
- moved OUT_MUL_3 1.10 mm to (136.0, 120.5)
- moved IN_B1 0.20 mm to (64.6, 113.0)
- renumbered OUT_ADD_OV to OUT_ADD_OV0
Routing:
- net IN_B2: track 38.5 -> 39.4 mm
- net /collector/OUT_2: track 17.3 -> 18.0 mm
- net OUT_MUL_3: track 41.1 -> 40.5 mm
